File: hardware/Letterbox_Sentinel.kicad_pcb (KiCad board)
At the start: 2 copper layers, 64 x 50 mm, 17 parts, among them J1 5.5x2.1mm CENTRE +, J2 XT60PW-F FEMALE, J3 IR TX FEMALE SOCKET, J4 IR RX FEMALE SOCKET, J5 BME280 FEMALE SOCKET, Q1 BC547 C-B-E, U1 TSR 1-2433 SOCKETED

Commit message: Updated all files and directories
Parts:
- removed D2: 1N5819 ADC CLAMP, Diode_THT:D_DO-41_SOD81_P10.16mm_Horizontal
- J1: footprint Connector_BarrelJack:BarrelJack_CUI_PJ-102AH_Horizontal -> Connector_BarrelJack:BarrelJack_GCT_DCJ200-10-A_Horizontal
- moved R4 10.2 mm to (98.1, 110.5), turned to 180 degrees
- moved R2 10.1 mm to (98.0, 100.5), turned to 180 degrees
- moved U1 1.46 mm to (83.0, 86.5)
- moved J1 0.70 mm to (69.5, 88.8)
- moved Q1 0.50 mm to (118.0, 104.0)
- renumbered J_WEMOS_L1 to 3.3v, J_WEMOS_R1 to 5v, J4 to S
Routing:
- net /BAT_SENSE_A0: track 41.4 -> 13.4 mm
- net /Q1_BASE: track 33.9 -> 37.7 mm
- net /+3V3: track 124.4 -> 126.7 mm
- net /VIN_PROTECTED: track 20.5 -> 21.1 mm
Other:
- board text added: "+"
- board text added: "-"
- board text added: "100k"
- board text added: "10k"
- board text added: "330k"
- board text added: "4.7k"
- board text added: "BME 280"
- board text added: "IN5819"
- board text added: "IR RX"
- board text added: "IR TX"
- board text added: "Letterbox Sentinel Rev 1.0 © Jeremy Younger 2026"
- board text added: "TSR"
- board text added: "USB"
- board text added: "VCC"
- board text added: "Wemos D1 R2 Mini"
- board text removed: "Jeremy Younger"
