File: hardware/Letterbox_Sentinel.kicad_sch (KiCad schematic)
At the start: 17 parts, among them J1 5.5x2.1mm CENTRE +, J2 XT60PW-F FEMALE, J3 IR TX FEMALE SOCKET, J4 IR RX FEMALE SOCKET, J5 BME280 FEMALE SOCKET, Q1 BC547 C-B-E, U1 TSR 1-2433 SOCKETED

Commit message: Updated all files and directories
Parts:
- removed D2: 1N5819 ADC CLAMP, Diode_THT:D_DO-41_SOD81_P10.16mm_Horizontal, symbol Letterbox:DIODE
Changed lines of the file:
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@@
 	(wire
 		(pts
-			(xy 64.77 114.3) (xy 69.92 115)
+			(xy 119.38 100.33) (xy 124.92 101.27)
 		)
 		(stroke
@@
 	(wire
 		(pts
-			(xy 82.55 114.3) (xy 80.08 115)
+			(xy 237.49 53.34) (xy 235.08 52.54)
 		)
 		(stroke
@@
 	(wire
 		(pts
-			(xy 119.38 100.33) (xy 124.92 101.27)
+			(xy 212.09 59.69) (xy 210.08 60)
 		)
 		(stroke
@@
 		)
 	)
-	(wire
-		(pts
-			(xy 237.49 53.34) (xy 235.08 52.54)
-		)
-		(stroke
-			(width 0)
-			(type default)
-		)
-	)
-	(wire
-		(pts
-			(xy 212.09 59.69) (xy 210.08 60)
-		)
-		(stroke
-			(width 0)
-			(type default)
-		)
-	)
 	(label "+5V"
 		(at 153.67 107.95 0)
@@
 	)
 	(label "GND"
-		(at 82.55 114.3 0)
-		(effects
-			(font
-				(size 1 1)
-			)
-		)
-	)
-	(label "GND"
 		(at 96.52 41.91 90)
 		(effects
@@
 	(label "+3V3"
 		(at 244.92 121.19 0)
-		(effects
-			(font
-				(size 1 1)
-			)
-		)
-	)
-	(label "BAT_SENSE_A0"
-		(at 64.77 114.3 0)
 		(effects
 			(font
@@
 		)
 		(instances
-			(project "Letterbox_Sentinel_REV1_9_FIXED"
+			(project "Letterbox_Sentinel"
 				(path "/e2625038-ab52-4ef0-a819-a349524c764c"
 					(reference "J2")
@@
 		)
 		(instances
-			(project "Letterbox_Sentinel_REV1_9_FIXED"
+			(project "Letterbox_Sentinel"
 				(path "/e2625038-ab52-4ef0-a819-a349524c764c"
 					(reference "J_WEMOS_R1")
@@
 		)
 		(instances
-			(project "Letterbox_Sentinel_REV1_9_FIXED"
+			(project "Letterbox_Sentinel"
 				(path "/e2625038-ab52-4ef0-a819-a349524c764c"
 					(reference "J_WEMOS_L1")
@@
 		)
 		(instances
-			(project "Letterbox_Sentinel_REV1_9_FIXED"
+			(project "Letterbox_Sentinel"
 				(path "/e2625038-ab52-4ef0-a819-a349524c764c"
 					(reference "D1")
@@
 		)
 		(instances
-			(project "Letterbox_Sentinel_REV1_9_FIXED"
+			(project "Letterbox_Sentinel"
 				(path "/e2625038-ab52-4ef0-a819-a349524c764c"
 					(reference "R4")
@@
 		)
 		(instances
-			(project "Letterbox_Sentinel_REV1_9_FIXED"
+			(project "Letterbox_Sentinel"
 				(path "/e2625038-ab52-4ef0-a819-a349524c764c"
 					(reference "U1")
@@
 		)
 		(instances
-			(project "Letterbox_Sentinel_REV1_9_FIXED"
+			(project "Letterbox_Sentinel"
 				(path "/e2625038-ab52-4ef0-a819-a349524c764c"
 					(reference "J1")
@@
 		)
 		(instances
-			(project "Letterbox_Sentinel_REV1_9_FIXED"
+			(project "Letterbox_Sentinel"
 				(path "/e2625038-ab52-4ef0-a819-a349524c764c"
 					(reference "J3")
@@
 		)
 		(instances
-			(project "Letterbox_Sentinel_REV1_9_FIXED"
+			(project "Letterbox_Sentinel"
 				(path "/e2625038-ab52-4ef0-a819-a349524c764c"
 					(reference "R1")
@@
 		)
 		(instances
-			(project "Letterbox_Sentinel_REV1_9_FIXED"
+			(project "Letterbox_Sentinel"
 				(path "/e2625038-ab52-4ef0-a819-a349524c764c"
 					(reference "J4")
@@
 		)
 		(instances
-			(project "Letterbox_Sentinel_REV1_9_FIXED"
+			(project "Letterbox_Sentinel"
 				(path "/e2625038-ab52-4ef0-a819-a349524c764c"
 					(reference "Q1")
@@
 		)
 		(instances
-			(project "Letterbox_Sentinel_REV1_9_FIXED"
+			(project "Letterbox_Sentinel"
 				(path "/e2625038-ab52-4ef0-a819-a349524c764c"
 					(reference "R5")
@@
 		)
 		(instances
-			(project "Letterbox_Sentinel_REV1_9_FIXED"
+			(project "Letterbox_Sentinel"
 				(path "/e2625038-ab52-4ef0-a819-a349524c764c"
 					(reference "C1")
@@
 		)
 		(instances
-			(project "Letterbox_Sentinel_REV1_9_FIXED"
+			(project "Letterbox_Sentinel"
 				(path "/e2625038-ab52-4ef0-a819-a349524c764c"
 					(reference "R3")
@@
 		)
 		(instances
-			(project "Letterbox_Sentinel_REV1_9_FIXED"
+			(project "Letterbox_Sentinel"
 				(path "/e2625038-ab52-4ef0-a819-a349524c764c"
 					(reference "R2")
@@
 		)
 		(instances
-			(project "Letterbox_Sentinel_REV1_9_FIXED"
+			(project "Letterbox_Sentinel"
 				(path "/e2625038-ab52-4ef0-a819-a349524c764c"
 					(reference "J5")
 					(unit 1)
 				)
-			)
-		)
-	)
-	(symbol
-		(lib_id "Letterbox:DIODE")
-		(at 75 115 0)
-		(unit 1)
-		(body_style 1)
-		(exclude_from_sim no)
-		(in_bom yes)
-		(on_board yes)
-		(in_pos_files yes)
-		(dnp no)
-		(property "Reference" "D2"
-			(at 74.93 111.76 0)
-			(show_name no)
-			(do_not_autoplace no)
-			(effects
-				(font
-					(size 1 1)
-				)
-			)
-		)
-		(property "Value" "1N5819 ADC CLAMP"
-			(at 75 120 0)
-			(show_name no)
-			(do_not_autoplace no)
-			(effects
-				(font
-					(size 1 1)
-				)
-			)
-		)
-		(property "Footprint" "Diode_THT:D_DO-41_SOD81_P10.16mm_Horizontal"
-			(at 75 115 0)
-			(hide yes)
-			(show_name no)
-			(do_not_autoplace no)
-			(effects
-				(font
-					(size 1 1)
-				)
-			)
-		)
-		(property "Datasheet" ""
-			(at 75 115 0)
-			(hide yes)
-			(show_name no)
-			(do_not_autoplace no)
-			(effects
-				(font
-					(size 1 1)
-				)
-			)
-		)
-		(property "Description" "Letterbox Sentinel Rev 1.6"
-			(at 75 115 0)
-			(hide yes)
-			(show_name no)
-			(do_not_autoplace no)
-			(effects
-				(font
-					(size 1 1)
-				)
-			)
-		)
-		(pin "1"
-		)
-		(pin "2"
-		)
-		(instances
-			(project "Letterbox_Sentinel_REV1_9_FIXED"
-				(path "/e2625038-ab52-4ef0-a819-a349524c764c"
-					(reference "D2")
-					(unit 1)
-				)
