File: hardware/xiao_esp32c6/Letterbox_Sentinel_C6.kicad_pcb (KiCad board)
At the start: 2 copper layers, 64 x 50 mm, 16 parts, among them J1 5.5x2.1mm CENTRE +, J2 XT60PW-F FEMALE, J3 IR TX FEMALE SOCKET, J4 IR RX FEMALE SOCKET, Q1 BC547 C-B-E, U1 TSR 1-2450 SOCKETED

Commit message: Use vertical XT60PB-M battery connector and JST-XH IR headers
Parts:
- J2: value XT60PW-F FEMALE -> XT60PB-M VERTICAL MALE; footprint LetterboxC6:AMASS_XT60PW-F_1x02_P7.20mm_Horizontal_J2 -> LetterboxC6:AMASS_XT60PB-M_1x02_P7.20mm_Vertical_J2
- J3: value IR TX FEMALE SOCKET -> JST-XH IR TX; footprint LetterboxC6:PinSocket_1x02_P2.54mm_Vertical_J3 -> LetterboxC6:JST_XH_B2B-XH-A_1x02_P2.50mm_Vertical_J3
- J4: value IR RX FEMALE SOCKET -> JST-XH IR RX; footprint LetterboxC6:PinSocket_1x03_P2.54mm_Vertical_J4 -> LetterboxC6:JST_XH_B3B-XH-A_1x03_P2.50mm_Vertical_J4
- moved J4 13.7 mm to (117.5, 112.0)
- moved J2 9.73 mm to (113.0, 84.5)
- moved J3 6.31 mm to (110.0, 94.0)
Connections:
- J3 pad 1: /IR_TX_SW_GND -> /+3V3
- J3 pad 2: /+3V3 -> /IR_TX_SW_GND
- J4 pad 1: /IR_RX_GPIO1 -> /+3V3
- J4 pad 3: /+3V3 -> /IR_RX_GPIO1
Routing:
- net /IR_RX_GPIO1: track 39.6 -> 26.6 mm
- net /GND: track 152.0 -> 164.7 mm
- net /BAT_RAW+: track 69.5 -> 79.4 mm
- net /+3V3: track 93.3 -> 99.8 mm
- net /IR_TX_SW_GND: track 10.8 -> 15.5 mm
- net /Q1_BASE: track 33.5 -> 30.0 mm
- net /BAT_SENSE_GPIO0: track 31.2 -> 33.7 mm
Other:
- board text added: "+"
- board text added: "-"
- board text added: "IR RX JST-XH"
- board text added: "IR TX JST-XH"
- board text added: "XT60PB-M"
- board text removed: "IR RX"
- board text removed: "IR TX"
