File: hardware/xiao_esp32c6/Letterbox_Sentinel_C6.kicad_sch (KiCad schematic)
At the start: 16 parts, among them J1 5.5x2.1mm CENTRE +, J2 XT60PW-F FEMALE, J3 IR TX FEMALE SOCKET, J4 IR RX FEMALE SOCKET, Q1 BC547 C-B-E, U1 TSR 1-2450 SOCKETED

Commit message: Use vertical XT60PB-M battery connector and JST-XH IR headers
Parts:
- J2: value XT60PW-F FEMALE -> XT60PB-M VERTICAL MALE; footprint LetterboxC6:AMASS_XT60PW-F_1x02_P7.20mm_Horizontal_J2 -> LetterboxC6:AMASS_XT60PB-M_1x02_P7.20mm_Vertical_J2
- J3: value IR TX FEMALE SOCKET -> JST-XH IR TX; footprint LetterboxC6:PinSocket_1x02_P2.54mm_Vertical_J3 -> LetterboxC6:JST_XH_B2B-XH-A_1x02_P2.50mm_Vertical_J3
- J4: value IR RX FEMALE SOCKET -> JST-XH IR RX; footprint LetterboxC6:PinSocket_1x03_P2.54mm_Vertical_J4 -> LetterboxC6:JST_XH_B3B-XH-A_1x03_P2.50mm_Vertical_J4
Connections:
- net +3V3: now also J3.1, J4.1; no longer J3.2, J4.3
- net IR_RX_GPIO1: now also J4.3; no longer J4.1
- net IR_TX_SW_GND: now also J3.2; no longer J3.1
